Commit message: finish cam imu gps

File: workspace/src/robot_startup/urdf/mogi_bot.xacro (robot description, xacro)
@@ -170,3 +170,11 @@
   <link name="camera_link_optical">
   </link>
+  <!-- IMU -->
+  <joint name="imu_joint" type="fixed">
+    <origin xyz="0 0 0" rpy="0 0 0" />
+    <parent link="base_link"/>
+    <child link="imu_link" />
+  </joint>
+  <link name="imu_link">
+  </link>
 </robot>

Commit message: finnish 2 sensor lesson

File: workspace/src/robot_startup/urdf/mogi_bot.xacro (robot description, xacro)
@@ -124,5 +124,5 @@
       <geometry>
         <!--cylinder radius=".1" length=".05"/-->
-        <mesh filename = "package://robot_startup/meshes/wheel.dae"/>
+        <mesh filename = "package://robot_startup/meshes/wheel.dae"></mesh>
       </geometry>
       <material name="green"/>
@@ -178,3 +178,33 @@
   <link name="imu_link">
   </link>
+  <!-- Lidar -->
+  <joint type="fixed" name="scan_joint">
+    <origin xyz="0.0 0 0.15" rpy="0 0 0"/>
+    <child link="scan_link"/>
+    <parent link="base_link"/>
+    <axis xyz="0 1 0" rpy="0 0 0"/>
+  </joint>
+  <link name='scan_link'>
+    <inertial>
+      <mass value="1e-5"/>
+      <origin xyz="0 0 0" rpy="0 0 0"/>
+      <inertia
+          ixx="1e-6" ixy="0" ixz="0"
+          iyy="1e-6" iyz="0"
+          izz="1e-6"
+      />
+    </inertial>
+    <collision name='collision'>
+      <origin xyz="0 0 0" rpy="0 0 0"/>
+      <geometry>
+        <box size=".1 .1 .1"/>
+      </geometry>
+    </collision>
+    <visual name='scan_link_visual'>
+      <origin xyz="0 0 0" rpy="0 0 0"/>
+      <geometry>
+        <mesh filename = "package://robot_startup/meshes/lidar.dae"/>
+      </geometry>
+    </visual>
+  </link>
 </robot>
