Commit message: add mapping and nav demo

File: workspace/src/pie_bringup/urdf/pie_bot.urdf.xacro (robot description, xacro)
@@ -10,5 +10,5 @@
   </joint>
   <link name="base_link">
-    <visual name='base_link_visual'>
+    <visual>
       <origin xyz="-0.032 0 0.0" rpy="0 0 0"/>
       <geometry>
@@ -17,5 +17,5 @@
       <material name="light_black"/>
     </visual>
-    <collision name='base_link_collision'>
+    <collision>
       <origin xyz="-0.032 0 0.070" rpy="0 0 0"/>
       <geometry>
@@ -31,5 +31,4 @@
     </inertial>
   </link>
-  <!-- Wheels -->
   <joint name="wheel_left_joint" type="continuous">
     <parent link="base_link"/>
@@ -37,9 +36,7 @@
     <origin xyz="0.0 0.08 0.023" rpy="-1.57 0 0"/>
     <axis xyz="0 0 1"/>
-    <limit effort="10000" velocity="1000"/>
-    <dynamics damping="1.0" friction="1.0"/>
   </joint>
   <link name="wheel_left_link">
-    <visual name='wheel_left_visual'>
+    <visual>
       <origin xyz="0 0 0" rpy="1.57 0 0"/>
       <geometry>
@@ -48,5 +45,5 @@
       <material name="dark"/>
     </visual>
-    <collision name='wheel_left_collision'>
+    <collision>
       <origin xyz="0 0 0" rpy="0 0 0"/>
       <geometry>
@@ -67,9 +64,7 @@
     <origin xyz="0.0 -0.080 0.023" rpy="-1.57 0 0"/>
     <axis xyz="0 0 1"/>
-    <limit effort="10000" velocity="1000"/>
-    <dynamics damping="1.0" friction="1.0"/>
   </joint>
   <link name="wheel_right_link">
-    <visual name='wheel_right__visual'>
+    <visual>
       <origin xyz="0 0 0" rpy="1.57 0 0"/>
       <geometry>
@@ -78,5 +73,5 @@
       <material name="dark"/>
     </visual>
-    <collision name='wheel_right_collision'>
+    <collision>
       <origin xyz="0 0 0" rpy="0 0 0"/>
       <geometry>
