Commit message: add rgbd camera plugin and xacro args

File: pie_bringup/urdf/camera.gazebo.xacro (robot description, xacro)
@@ -1,4 +1,5 @@
 <?xml version="1.0"?>
 <robot name="rgb_camera" xmlns:xacro="http://ros.org/wiki/xacro">
+    <xacro:arg name="camera_visual"  default="false"/>
     <gazebo reference="camera_link">
         <sensor type="camera" name="camera">
@@ -28,6 +29,6 @@
             <alwaysOn>true</alwaysOn>
             <updateRate>0.0</updateRate>
-            <cameraName>camera</cameraName>
-            <imageTopicName>image</imageTopicName>
+            <cameraName>rgb_camera</cameraName>
+            <imageTopicName>rgb/image_raw</imageTopicName>
             <cameraInfoTopicName>camera_info</cameraInfoTopicName>
             <frameName>camera_link_optical</frameName>

File: pie_bringup/urdf/pie_bot.urdf.xacro (robot description, xacro)
@@ -4,6 +4,10 @@
   <xacro:include filename="$(find pie_bringup)/urdf/pie_bot.gazebo.xacro"/>
   <xacro:arg name="use_camera"  default="false"/>
+  <xacro:arg name="use_rgbd_camera"  default="false"/>
   <xacro:if value="$(arg use_camera)">
     <xacro:include filename="$(find pie_bringup)/urdf/camera.urdf.xacro"/>
+  </xacro:if>
+  <xacro:if value="$(arg use_rgbd_camera)">
+    <xacro:include filename="$(find pie_bringup)/urdf/rgbd_camera.urdf.xacro"/>
   </xacro:if>
   <link name="base_footprint"/>

File: pie_bringup/urdf/rgbd_camera.urdf.xacro (robot description, xacro)
@@ -1,12 +1,12 @@
 <?xml version="1.0" ?>
-<robot name="rgb_camera" xmlns:xacro="http://ros.org/wiki/xacro">
-  <xacro:include filename="$(find pie_bringup)/urdf/camera.gazebo.xacro"/>
-    <joint type="fixed" name="camera_joint">
+<robot name="rgbd_camera" xmlns:xacro="http://ros.org/wiki/xacro">
+  <xacro:include filename="$(find pie_bringup)/urdf/rgbd_camera.gazebo.xacro"/>
+    <joint type="fixed" name="rgbd_camera_joint">
         <origin xyz="0.03 0 0.071" rpy="0 -0.52 0"/>
-        <child link="camera_link"/>
+        <child link="rgbd_camera_link"/>
         <parent link="base_link"/>
         <axis xyz="0 1 0" />
     </joint>
-    <link name='camera_link'>
+    <link name='rgbd_camera_link'>
         <pose>0 0 0 0 0 0</pose>
         <inertial>
@@ -19,5 +19,5 @@
             />
         </inertial>
-        <collision name='collision'>
+        <collision name='rgbd_camera_collision'>
             <origin xyz="0 0 0" rpy="0 0 0"/>
             <geometry>
@@ -25,5 +25,5 @@
             </geometry>
         </collision>
-        <visual name='camera_link_visual'>
+        <visual name='rgbd_camera_link_visual'>
             <origin xyz="0 0 0" rpy="0 0 0"/>
             <geometry>

Commit message: fix camera nameing

File: pie_bringup/urdf/camera.gazebo.xacro (robot description, xacro)
@@ -2,5 +2,5 @@
 <robot name="rgb_camera" xmlns:xacro="http://ros.org/wiki/xacro">
     <xacro:arg name="camera_visual"  default="false"/>
-    <gazebo reference="camera_link">
+    <gazebo reference="rgb_camera_link">
         <sensor type="camera" name="camera">
             <update_rate>30.0</update_rate>
@@ -31,6 +31,6 @@
             <cameraName>rgb_camera</cameraName>
             <imageTopicName>rgb/image_raw</imageTopicName>
-            <cameraInfoTopicName>camera_info</cameraInfoTopicName>
-            <frameName>camera_link_optical</frameName>
+            <cameraInfoTopicName>rgb/camera_info</cameraInfoTopicName>
+            <frameName>rgb_camera_link</frameName>
             <hackBaseline>0.0</hackBaseline>
             <distortionK1>0.0</distortionK1>

File: pie_bringup/urdf/camera.urdf.xacro (robot description, xacro)
@@ -4,9 +4,9 @@
     <joint type="fixed" name="camera_joint">
         <origin xyz="0.03 0 0.071" rpy="0 -0.52 0"/>
-        <child link="camera_link"/>
+        <child link="rgb_camera_link"/>
         <parent link="base_link"/>
         <axis xyz="0 1 0" />
     </joint>
-    <link name='camera_link'>
+    <link name='rgb_camera_link'>
         <pose>0 0 0 0 0 0</pose>
         <inertial>

File: pie_bringup/urdf/rgbd_camera.gazebo.xacro (robot description, xacro)
@@ -28,5 +28,5 @@
         <depthImageTopicName>depth/image_raw</depthImageTopicName>
         <pointCloudTopicName>depth/points</pointCloudTopicName>
-        <cameraInfoTopicName>camera_info</cameraInfoTopicName>
+        <cameraInfoTopicName>rgb/camera_info</cameraInfoTopicName>
         <depthImageCameraInfoTopicName>depth/camera_info</depthImageCameraInfoTopicName>
         <pointCloudCutoff>0.5</pointCloudCutoff>
