Commit message: change robot inertias

File: pie_bringup/urdf/pie_bot.urdf.xacro (robot description, xacro)
@@ -33,8 +33,8 @@
     <inertial>
       <origin xyz="0 0 0" rpy="0 0 0"/>
-      <mass value="8.2573504e-01"/>
-      <inertia ixx="2.2124416e-03" ixy="-1.2294101e-05" ixz="3.4938785e-05"
-               iyy="2.1193702e-03" iyz="-5.0120904e-06"
-               izz="2.0064271e-03" />
+      <mass value="1.0"/>
+      <inertia ixx="0.001" ixy="0.000" ixz="0.000"
+               iyy="0.001" iyz="0.000"
+               izz="0.001" />
     </inertial>
   </link>
@@ -62,7 +62,7 @@
       <origin xyz="0 0 0" />
       <mass value="2.8498940e-02" />
-      <inertia ixx="1.1175580e-05" ixy="-4.2369783e-11" ixz="-5.9381719e-09"
-               iyy="1.1192413e-05" iyz="-1.4400107e-11"
-               izz="2.0712558e-05" />
+      <inertia ixx="1.8158194e-03" ixy="-9.3392e-12" ixz="1.04909e-11"
+               iyy="3.2922126e-03" iyz="5.75694e-11"
+               izz="1.8158194e-03" />
       </inertial>
   </link>
@@ -90,7 +90,7 @@
       <origin xyz="0 0 0" />
       <mass value="2.8498940e-02" />
-      <inertia ixx="1.1175580e-05" ixy="-4.2369783e-11" ixz="-5.9381719e-09"
-               iyy="1.1192413e-05" iyz="-1.4400107e-11"
-               izz="2.0712558e-05" />
+      <inertia ixx="1.8158194e-03" ixy="-9.3392e-12" ixz="1.04909e-11"
+               iyy="3.2922126e-03" iyz="5.75694e-11"
+               izz="1.8158194e-03" />
       </inertial>
   </link>

Commit message: reduca camera angle

File: pie_bringup/urdf/pie_bot.urdf.xacro (robot description, xacro)
@@ -5,4 +5,5 @@
   <xacro:arg name="use_camera"  default="false"/>
   <xacro:arg name="use_rgbd_camera"  default="false"/>
+<!-- https://github.com/ROBOTIS-GIT/turtlebot3_simulations/blob/8241af04a4e56e656d4be24a5c3971e3359bf751/turtlebot3_gazebo/models/turtlebot3_burger/model.sdf#L146 -->
   <xacro:if value="$(arg use_camera)">
     <xacro:include filename="$(find pie_bringup)/urdf/camera.urdf.xacro"/>

File: pie_bringup/urdf/rgbd_camera.urdf.xacro (robot description, xacro)
@@ -3,5 +3,5 @@
   <xacro:include filename="$(find pie_bringup)/urdf/rgbd_camera.gazebo.xacro"/>
     <joint type="fixed" name="rgbd_camera_joint">
-        <origin xyz="0.03 0 0.071" rpy="0 -0.52 0"/>
+        <origin xyz="0.03 0 0.071" rpy="0 -0.35 0"/>
         <child link="rgbd_camera_link"/>
         <parent link="base_link"/>

Commit message: launch and urdf improvements

File: pie_bringup/urdf/pie_bot.urdf.xacro (robot description, xacro)
@@ -34,8 +34,8 @@
     <inertial>
       <origin xyz="0 0 0" rpy="0 0 0"/>
-      <mass value="1.0"/>
-      <inertia ixx="0.001" ixy="0.000" ixz="0.000"
-               iyy="0.001" iyz="0.000"
-               izz="0.001" />
+      <mass value="8.2573504e-01"/>
+      <inertia ixx="2.2124416e-03" ixy="-1.2294101e-05" ixz="3.4938785e-05"
+               iyy="2.1193702e-03" iyz="-5.0120904e-06"
+               izz="2.0064271e-03" />
     </inertial>
   </link>
@@ -59,12 +59,24 @@
         <cylinder length="0.018" radius="0.033"/>
       </geometry>
+      <surface>
+        <friction>
+          <ode>
+            <mu>100000.0</mu>
+            <mu2>100000.0</mu2>
+          </ode>
+        </friction>
+      </surface>
     </collision>
     <inertial>
       <origin xyz="0 0 0" />
       <mass value="2.8498940e-02" />
-      <inertia ixx="1.8158194e-03" ixy="-9.3392e-12" ixz="1.04909e-11"
+      <inertia ixx="1.1175580e-05" ixy="-4.2369783e-11" ixz="-5.9381719e-09"
+               iyy="1.1192413e-05" iyz="-1.4400107e-11"
+               izz="2.0712558e-05" />
+      </inertial>
+      <!-- <inertia ixx="1.8158194e-03" ixy="-9.3392e-12" ixz="1.04909e-11"
                iyy="3.2922126e-03" iyz="5.75694e-11"
                izz="1.8158194e-03" />
-      </inertial>
+      </inertial> -->
   </link>
   <joint name="wheel_right_joint" type="continuous">
@@ -87,12 +99,24 @@
         <cylinder length="0.018" radius="0.033"/>
       </geometry>
+      <surface>
+        <friction>
+          <ode>
+            <mu>100000.0</mu>
+            <mu2>100000.0</mu2>
+          </ode>
+        </friction>
+      </surface>
     </collision>
     <inertial>
       <origin xyz="0 0 0" />
       <mass value="2.8498940e-02" />
-      <inertia ixx="1.8158194e-03" ixy="-9.3392e-12" ixz="1.04909e-11"
+      <inertia ixx="1.1175580e-05" ixy="-4.2369783e-11" ixz="-5.9381719e-09"
+               iyy="1.1192413e-05" iyz="-1.4400107e-11"
+               izz="2.0712558e-05" />
+      </inertial>
+      <!-- <inertia ixx="1.8158194e-03" ixy="-9.3392e-12" ixz="1.04909e-11"
                iyy="3.2922126e-03" iyz="5.75694e-11"
                izz="1.8158194e-03" />
-      </inertial>
+      </inertial> -->
   </link>
   <joint name="caster_back_joint" type="fixed">

Commit message: Improvements (#13)
* change robot inertias

* add option to start gazebo gui

* reduca camera angle

* make subms http instead ssh for virgins

* remove subms

* subms via http

* remove subms2

* launch and urdf improvements

* add test subm

* add all subms

File: pie_bringup/urdf/pie_bot.urdf.xacro (robot description, xacro)
@@ -5,4 +5,5 @@
   <xacro:arg name="use_camera"  default="false"/>
   <xacro:arg name="use_rgbd_camera"  default="false"/>
+<!-- https://github.com/ROBOTIS-GIT/turtlebot3_simulations/blob/8241af04a4e56e656d4be24a5c3971e3359bf751/turtlebot3_gazebo/models/turtlebot3_burger/model.sdf#L146 -->
   <xacro:if value="$(arg use_camera)">
     <xacro:include filename="$(find pie_bringup)/urdf/camera.urdf.xacro"/>
@@ -58,4 +59,12 @@
         <cylinder length="0.018" radius="0.033"/>
       </geometry>
+      <surface>
+        <friction>
+          <ode>
+            <mu>100000.0</mu>
+            <mu2>100000.0</mu2>
+          </ode>
+        </friction>
+      </surface>
     </collision>
     <inertial>
@@ -66,4 +75,8 @@
                izz="2.0712558e-05" />
       </inertial>
+      <!-- <inertia ixx="1.8158194e-03" ixy="-9.3392e-12" ixz="1.04909e-11"
+               iyy="3.2922126e-03" iyz="5.75694e-11"
+               izz="1.8158194e-03" />
+      </inertial> -->
   </link>
   <joint name="wheel_right_joint" type="continuous">
@@ -86,4 +99,12 @@
         <cylinder length="0.018" radius="0.033"/>
       </geometry>
+      <surface>
+        <friction>
+          <ode>
+            <mu>100000.0</mu>
+            <mu2>100000.0</mu2>
+          </ode>
+        </friction>
+      </surface>
     </collision>
     <inertial>
@@ -94,4 +115,8 @@
                izz="2.0712558e-05" />
       </inertial>
+      <!-- <inertia ixx="1.8158194e-03" ixy="-9.3392e-12" ixz="1.04909e-11"
+               iyy="3.2922126e-03" iyz="5.75694e-11"
+               izz="1.8158194e-03" />
+      </inertial> -->
   </link>
   <joint name="caster_back_joint" type="fixed">
